File: atx040-main-pcb.kicad_pcb (KiCad board)
At the start: 4 copper layers, 243.8 x 170.2 mm, 12 parts, among them J200 ATX20P, J400 C96, U100 MC68040RC, U102 W25Q80D, U300 SIMM72, U301 SIMM72

Commit message: Finished board + fab files
Parts:
- removed J400: C96, connector:C96ABCM
- removed U102: W25Q80D, Package_SO:SOIC-8_3.9x4.9mm_P1.27mm
- added BT600: Battery_Cell, Battery:BatteryHolder_Keystone_1060_1x2032, F.Cu at (181.6, 180.3)
- added C100: 100nF, Capacitor_SMD:C_0603_1608Metric, B.Cu at (152.2, 92.5)
- added C101: 100nF, Capacitor_SMD:C_0603_1608Metric, B.Cu at (152.2, 98.0)
- added C102: 100nF, Capacitor_SMD:C_0603_1608Metric, B.Cu at (152.2, 79.0)
- added C103: 100nF, Capacitor_SMD:C_0603_1608Metric, B.Cu at (152.2, 73.5)
- added C104: 100nF, Capacitor_SMD:C_0603_1608Metric, B.Cu at (152.2, 60.0)
- added C105: 100nF, Capacitor_SMD:C_0603_1608Metric, B.Cu at (152.2, 54.2)
- added C110: 100nF, Capacitor_SMD:C_0603_1608Metric, B.Cu at (216.7, 77.5)
- added C111: 100nF, Capacitor_SMD:C_0603_1608Metric, B.Cu at (210.8, 52.1)
- added C112: 100nF, Capacitor_SMD:C_0603_1608Metric, B.Cu at (188.2, 51.1)
- added C113: 100nF, Capacitor_SMD:C_0603_1608Metric, B.Cu at (189.5, 78.5)
- added C114: 100nF, Capacitor_SMD:C_0603_1608Metric, B.Cu at (203.2, 90.2)
- added C115: 100nF, Capacitor_SMD:C_0603_1608Metric, B.Cu at (177.5, 94.0)
- added C116: 100uF, Capacitor_SMD:C_1206_3216Metric, B.Cu at (202.4, 76.2)
- added C117: 4.7uF, Capacitor_SMD:C_0805_2012Metric, B.Cu at (177.0, 69.8)
- added C118: 4.7uF, Capacitor_SMD:C_0805_2012Metric, B.Cu at (227.3, 68.8)
- added C200: 4.7uF, Capacitor_SMD:C_0805_2012Metric, F.Cu at (142.5, 126.0)
- added C201: 4.7uF, Capacitor_SMD:C_0805_2012Metric, F.Cu at (142.5, 121.0)
- added C202: 4.7uF, Capacitor_SMD:C_0805_2012Metric, F.Cu at (140.2, 126.0)
- added C203: 4.7uF, Capacitor_SMD:C_0805_2012Metric, F.Cu at (144.8, 121.0)
- added C204: 4.7uF, Capacitor_SMD:C_0805_2012Metric, F.Cu at (140.2, 121.0)
- added C205: 0.47uF, Capacitor_SMD:C_0402_1005Metric, B.Cu at (125.5, 122.2)
- added C210: 100uF, Capacitor_SMD:C_1206_3216Metric, F.Cu at (153.0, 131.0)
- added C211: 100uF, Capacitor_SMD:C_1206_3216Metric, F.Cu at (153.0, 133.5)
- added C212: 100uF, Capacitor_SMD:C_1206_3216Metric, F.Cu at (153.0, 117.5)
- added C213: 100uF, Capacitor_SMD:C_1206_3216Metric, F.Cu at (153.0, 115.0)
- added C214: 100uF, Capacitor_SMD:C_1206_3216Metric, F.Cu at (153.0, 112.5)
- added C215: 4.7uF, Capacitor_SMD:C_0805_2012Metric, F.Cu at (114.0, 135.0)
- added C216: 4.7uF, Capacitor_SMD:C_0805_2012Metric, F.Cu at (136.0, 135.0)
- added C217: 4.7uF, Capacitor_SMD:C_0805_2012Metric, F.Cu at (114.0, 113.0)
- added C218: 4.7uF, Capacitor_SMD:C_0805_2012Metric, F.Cu at (136.0, 113.0)
- added C219: 4.7uF, Capacitor_SMD:C_0805_2012Metric, B.Cu at (128.2, 124.2)
- added C220: 0.47uF, Capacitor_SMD:C_0402_1005Metric, B.Cu at (130.5, 125.2)
- added C221: 0.47uF, Capacitor_SMD:C_0402_1005Metric, B.Cu at (120.8, 129.5)
- added C222: 0.47uF, Capacitor_SMD:C_0402_1005Metric, B.Cu at (130.8, 129.5)
- added C223: 0.47uF, Capacitor_SMD:C_0402_1005Metric, B.Cu at (126.8, 120.5)
- added C224: 0.47uF, Capacitor_SMD:C_0402_1005Metric, B.Cu at (130.5, 119.2)
- added C225: 0.47uF, Capacitor_SMD:C_0402_1005Metric, B.Cu at (119.5, 118.2)
- added C226: 0.47uF, Capacitor_SMD:C_0402_1005Metric, B.Cu at (121.5, 123.2)
- added C227: 0.47uF, Capacitor_SMD:C_0402_1005Metric, B.Cu at (122.5, 126.8)
- added C230: 100nF, Capacitor_SMD:C_0402_1005Metric, B.Cu at (136.2, 144.2)
- added C240: 100nF, Capacitor_SMD:C_0402_1005Metric, B.Cu at (146.0, 130.8)
- added C300: 4.7uF, Capacitor_SMD:C_0805_2012Metric, F.Cu at (165.5, 124.0)
- added C301: 4.7uF, Capacitor_SMD:C_0805_2012Metric, F.Cu at (144.8, 126.0)
- added C302: 100nF, Capacitor_SMD:C_0603_1608Metric, F.Cu at (257.8, 100.3)
- added C303: 100nF, Capacitor_SMD:C_0603_1608Metric, F.Cu at (233.2, 106.4)
- added C304: 100nF, Capacitor_SMD:C_0603_1608Metric, F.Cu at (230.1, 112.5)
- added C400: 100nF, Capacitor_SMD:C_0603_1608Metric, F.Cu at (99.3, 132.1)
- added C401: 100nF, Capacitor_SMD:C_0603_1608Metric, F.Cu at (92.2, 132.1)
- added C402: 100nF, Capacitor_SMD:C_0603_1608Metric, F.Cu at (92.2, 115.8)
- added C403: 100nF, Capacitor_SMD:C_0603_1608Metric, F.Cu at (99.3, 115.8)
- added C404: 100nF, Capacitor_SMD:C_0603_1608Metric, F.Cu at (89.4, 133.1)
- added C405: 100nF, Capacitor_SMD:C_0603_1608Metric, F.Cu at (96.0, 133.1)
- added C406: 100nF, Capacitor_SMD:C_0603_1608Metric, F.Cu at (110.5, 133.1)
- added C500: 100nF, Capacitor_SMD:C_0603_1608Metric, F.Cu at (60.3, 154.9)
- added C501: 100nF, Capacitor_SMD:C_0603_1608Metric, F.Cu at (63.5, 154.9)
- added C502: 100nF, Capacitor_SMD:C_0603_1608Metric, B.Cu at (74.9, 145.3)
- added C503: 100nF, Capacitor_SMD:C_0603_1608Metric, B.Cu at (68.8, 154.2)
- added C504: 100nF, Capacitor_SMD:C_0603_1608Metric, B.Cu at (68.8, 147.8)
- added C600: 100nF, Capacitor_SMD:C_0603_1608Metric, B.Cu at (36.2, 175.3)
- added C601: 100nF, Capacitor_SMD:C_0603_1608Metric, B.Cu at (158.1, 155.4)
- added C602: 100nF, Capacitor_SMD:C_0603_1608Metric, B.Cu at (175.3, 144.8)
- added J200: JTAG, Connector_PinHeader_2.54mm:PinHeader_1x06_P2.54mm_Vertical, F.Cu at (136.4, 96.0)
- added J201: UART, Connector_PinHeader_2.54mm:PinHeader_1x03_P2.54mm_Vertical, F.Cu at (79.4, 119.4)
- added J301: PWR_SW, Connector_PinHeader_2.54mm:PinHeader_1x02_P2.54mm_Vertical, F.Cu at (226.1, 194.3)
- added J302: PWR_LED, Connector_PinHeader_2.54mm:PinHeader_1x02_P2.54mm_Vertical, F.Cu at (248.9, 194.3)
- added J303: RST_SW, Connector_PinHeader_2.54mm:PinHeader_1x02_P2.54mm_Vertical, F.Cu at (233.7, 194.3)
- added J304: HDD_LED, Connector_PinHeader_2.54mm:PinHeader_1x02_P2.54mm_Vertical, F.Cu at (241.3, 194.3)
- added J305: ISP, Connector_PinHeader_2.54mm:PinHeader_2x05_P2.54mm_Vertical, F.Cu at (238.8, 113.0)
- added J500: VGA, Connector_Dsub:DSUB-15-HD_Female_Horizontal_P2.29x1.98mm_EdgePinOffset3.03mm_Housed_MountingHolesOffset4.94mm, F.Cu at (39.4, 153.7)
- added J600: Micro_SD_Card_Det, Connector_Card:microSD_HC_Molex_104031-0811, F.Cu at (39.0, 176.5)
- added J610: Conn_01x06, Connector_PinSocket_2.54mm:PinSocket_1x06_P2.54mm_Vertical, F.Cu at (59.7, 129.5)
- added J611: Conn_01x09, Connector_PinSocket_2.54mm:PinSocket_1x09_P2.54mm_Vertical, F.Cu at (62.2, 109.2)
- added J620: Conn_01x05, Connector_PinSocket_2.54mm:PinSocket_1x05_P2.54mm_Vertical, F.Cu at (36.8, 101.6)
- added J621: Conn_01x05, Connector_PinSocket_2.54mm:PinSocket_1x05_P2.54mm_Vertical, F.Cu at (36.8, 80.0)
- added J630: PS2, connector:KMDTX-HT-6S-BSC, F.Cu at (32.0, 66.8)
- added J640: USB, Connector_PinHeader_2.54mm:PinHeader_2x05_P2.54mm_Vertical, F.Cu at (180.3, 121.9)
- added M600: Fan_PC_Chassis, Connector:FanPinHeader_1x03_P2.54mm_Vertical, F.Cu at (248.9, 54.6)
- added M601: Fan_PC_Chassis, Connector:FanPinHeader_1x03_P2.54mm_Vertical, F.Cu at (248.9, 63.5)
- added M602: Fan_PC_Chassis, Connector:FanPinHeader_1x03_P2.54mm_Vertical, F.Cu at (248.9, 72.4)
- added R100: 4K7, Resistor_SMD:R_0603_1608Metric, F.Cu at (231.4, 57.1)
- added R200: 330R, Resistor_SMD:R_0603_1608Metric, B.Cu at (132.2, 133.0)
- added R201: 4K7, Resistor_SMD:R_0603_1608Metric, B.Cu at (110.5, 132.7)
- added R202: 100R, Resistor_SMD:R_0603_1608Metric, F.Cu at (129.8, 140.8)
- added R203: 100R, Resistor_SMD:R_0603_1608Metric, F.Cu at (128.2, 139.2)
- added R204: 4K7, Resistor_SMD:R_0603_1608Metric, F.Cu at (130.8, 149.6)
- added R205: 4K7, Resistor_SMD:R_0603_1608Metric, F.Cu at (135.5, 147.5)
- added R206: 4K7, Resistor_SMD:R_0603_1608Metric, F.Cu at (125.7, 146.1)
- added R207: 4K7, Resistor_SMD:R_0603_1608Metric, B.Cu at (113.7, 131.4)
- added R209: 100R, Resistor_SMD:R_0402_1005Metric, F.Cu at (137.0, 118.5)
- added R210: 100R, Resistor_SMD:R_0402_1005Metric, F.Cu at (138.0, 119.5)
- added R211: 100R, Resistor_SMD:R_0402_1005Metric, F.Cu at (113.0, 116.1)
- added R212: 330R, Resistor_SMD:R_0402_1005Metric, F.Cu at (85.8, 124.5)
- added R213: 330R, Resistor_SMD:R_0402_1005Metric, F.Cu at (85.8, 123.0)
- added R214: 100R, Resistor_SMD:R_0402_1005Metric, F.Cu at (116.2, 137.2)
- added R215: 100R, Resistor_SMD:R_0402_1005Metric, B.Cu at (128.8, 134.2)
- added R216: 100R, Resistor_SMD:R_0402_1005Metric, F.Cu at (134.8, 138.0)
- added R217: 100R, Resistor_SMD:R_0402_1005Metric, F.Cu at (127.8, 135.0)
- added R300: 1K5, Resistor_SMD:R_0603_1608Metric, F.Cu at (248.9, 188.0)
- added R301: 1K5, Resistor_SMD:R_0603_1608Metric, F.Cu at (241.3, 188.0)
- added R302: 1K5, Resistor_SMD:R_0603_1608Metric, F.Cu at (241.3, 100.3)
- added R500: 560R, Resistor_SMD:R_0402_1005Metric, F.Cu at (69.2, 157.0)
- added R501: 75R, Resistor_SMD:R_0603_1608Metric, F.Cu at (56.6, 152.4)
- added R502: 75R, Resistor_SMD:R_0603_1608Metric, F.Cu at (58.4, 151.4)
- added R503: 75R, Resistor_SMD:R_0603_1608Metric, F.Cu at (58.4, 147.8)
- added R630: 4K7, Resistor_SMD:R_0603_1608Metric, F.Cu at (45.5, 66.0)
- added R631: 4K7, Resistor_SMD:R_0603_1608Metric, F.Cu at (45.5, 62.2)
- added R640: 22R, Resistor_SMD:R_0603_1608Metric, F.Cu at (175.3, 127.0)
- added R641: 1K5, Resistor_SMD:R_0603_1608Metric, F.Cu at (177.8, 129.5)
- added R642: 22R, Resistor_SMD:R_0603_1608Metric, F.Cu at (175.3, 124.5)
- added R643: 22R, Resistor_SMD:R_0603_1608Metric, F.Cu at (188.0, 127.0)
- added R644: 1K5, Resistor_SMD:R_0603_1608Metric, F.Cu at (185.4, 129.5)
- added R645: 22R, Resistor_SMD:R_0603_1608Metric, F.Cu at (188.0, 124.5)
- added R650: 1K5, Resistor_SMD:R_0603_1608Metric, F.Cu at (151.1, 149.9)
- added R651: 1K5, Resistor_SMD:R_0603_1608Metric, F.Cu at (151.1, 153.0)
- added U110: MC74LCX16245, Package_SO:TSSOP-48_6.1x12.5mm_P0.5mm, F.Cu at (152.4, 76.2)
- added U111: MC74LCX16245, Package_SO:TSSOP-48_6.1x12.5mm_P0.5mm, F.Cu at (152.4, 57.1)
- added U120: MC74LCX16245, Package_SO:TSSOP-48_6.1x12.5mm_P0.5mm, F.Cu at (152.4, 95.2)
- added U200: XC6SLX16-FTG256, Package_BGA:Xilinx_FTG256, F.Cu at (125.0, 124.0)
- added U201: W25Q80D, Package_SO:SOIC-8_3.9x4.9mm_P1.27mm, F.Cu at (130.8, 146.1)
- added U302: TXB0102DCU, Package_SO:VSSOP-8_2.4x2.1mm_P0.5mm, F.Cu at (231.6, 109.5)
- added U400: W9825G6KH, Package_SO:TSOP-II-54_22.2x10.16mm_P0.8mm, F.Cu at (100.0, 124.1)
- added U500: ADV7123, Package_QFP:LQFP-48_7x7mm_P0.5mm, F.Cu at (70.5, 149.9)
- added U600: DS3231M, Package_SO:SOIC-16W_7.5x10.3mm_P1.27mm, F.Cu at (161.3, 154.9)
- added U601: CAT24C256, Package_SO:SOIC-8_3.9x4.9mm_P1.27mm, F.Cu at (175.3, 144.8)
- added X200: XO53, Oscillator:Oscillator_SMD_EuroQuartz_XO53-4Pin_5.0x3.2mm, F.Cu at (146.1, 130.8)
- U300: value SIMM72 -> AZ1117-1.2; footprint connector:SIM72 -> Package_TO_SOT_SMD:TO-252-2
- U301: value SIMM72 -> ATtiny2313A-PU; footprint connector:SIM72 -> Package_DIP:DIP-20_W7.62mm
- moved U301 112.7 mm to (246.4, 100.3)
- moved U100 91.6 mm to (203.2, 76.2), turned to 90 degrees
- moved U300 43.5 mm to (156.0, 124.0), turned to 180 degrees
- renumbered J200 to J300
Connections:
- net BR renamed Net-(U100-PadT18)
- net RSTI renamed /MC68040/TTL_RSTI
- net TM0 renamed Net-(U100-PadN18)
- net TM1 renamed Net-(U100-PadM18)
- net TM2 renamed Net-(U100-PadK17)
- U100 pad A1: AD31 -> /MC68040/TTL_AD3
- U100 pad A10: AD12 -> /MC68040/TTL_AD12
- U100 pad A11: AD13 -> /MC68040/TTL_AD13
- U100 pad A12: AD14 -> /MC68040/TTL_AD14
- U100 pad A13: AD15 -> /MC68040/TTL_AD15
- U100 pad A14: AD17 -> /MC68040/TTL_AD17
- U100 pad A15: AD19 -> /MC68040/TTL_AD19
- U100 pad A16: AD20 -> /MC68040/TTL_AD20
- U100 pad A17: AD21 -> /MC68040/TTL_AD21
- U100 pad A18: AD24 -> /MC68040/TTL_AD24
- U100 pad A2: AD3 -> /MC68040/TTL_AD3
- U100 pad A3: AD4 -> /MC68040/TTL_AD4
- U100 pad A4: AD5 -> /MC68040/TTL_AD5
- U100 pad A5: AD6 -> /MC68040/TTL_AD6
- U100 pad A6: AD7 -> /MC68040/TTL_AD7
- U100 pad A7: AD9 -> /MC68040/TTL_AD9
- U100 pad A8: AD10 -> /MC68040/TTL_AD10
- U100 pad A9: AD11 -> /MC68040/TTL_AD11
- U100 pad B1: AD29 -> /MC68040/TTL_AD4
- U100 pad B11: AD16 -> /MC68040/TTL_AD16
- U100 pad B12: AD18 -> /MC68040/TTL_AD18
- U100 pad B16: AD22 -> /MC68040/TTL_AD22
- U100 pad B18: AD26 -> /MC68040/TTL_AD26
- U100 pad B3: AD1 -> /MC68040/TTL_AD1
- U100 pad B7: AD8 -> /MC68040/TTL_AD8
- U100 pad C1: AD27 -> /MC68040/TTL_AD1
- U100 pad C15: AD23 -> /MC68040/TTL_AD23
- U100 pad C16: AD25 -> /MC68040/TTL_AD25
- U100 pad C18: AD28 -> /MC68040/TTL_AD28
- U100 pad C3: AD0 -> /MC68040/TTL_AD0
- U100 pad C4: AD2 -> /MC68040/TTL_AD2
- U100 pad D1: AD24 -> /MC68040/TTL_AD0
- U100 pad D16: AD27 -> /MC68040/TTL_AD27
- U100 pad D18: AD31 -> /MC68040/TTL_AD31
- U100 pad D3: AD30 -> /MC68040/TTL_AD2
- U100 pad E1: AD22 -> /MC68040/TTL_AD5
- U100 pad E16: AD29 -> /MC68040/TTL_AD29
- U100 pad E17: AD30 -> /MC68040/TTL_AD30
- U100 pad E18: AD8 -> /MC68040/TTL_AD31
- U100 pad E2: AD26 -> /MC68040/TTL_AD6
- U100 pad E3: AD28 -> /MC68040/TTL_AD7
- U100 pad F1: AD21 -> /MC68040/TTL_AD8
- U100 pad F16: AD9 -> /MC68040/TTL_AD29
- U100 pad F18: AD7 -> /MC68040/TTL_AD30
- U100 pad F3: AD25 -> /MC68040/TTL_AD9
- U100 pad G1: AD20 -> /MC68040/TTL_AD10
- U100 pad G16: AD6 -> /MC68040/TTL_AD27
- U100 pad G18: AD5 -> /MC68040/TTL_AD28
- U100 pad G3: AD23 -> /MC68040/TTL_AD11
- U100 pad H1: AD18 -> /MC68040/TTL_AD12
- U100 pad H18: AD4 -> /MC68040/TTL_AD26
- U100 pad J1: AD17 -> /MC68040/TTL_AD13
- U100 pad J17: AD2 -> /MC68040/TTL_AD25
- U100 pad J18: AD3 -> /MC68040/TTL_AD24
- U100 pad J2: AD19 -> /MC68040/TTL_AD16
- U100 pad K1: AD15 -> /MC68040/TTL_AD14
- U100 pad K18: AD1 -> /MC68040/TTL_AD22
- U100 pad K2: AD16 -> /MC68040/TTL_AD18
- U100 pad L1: AD14 -> /MC68040/TTL_AD15
- U100 pad L18: AD0 -> /MC68040/TTL_AD23
- U100 pad M1: AD13 -> /MC68040/TTL_AD17
- U100 pad N1: AD12 -> /MC68040/TTL_AD19
- U100 pad N16: RW -> /MC68040/TTL_RW
- U100 pad N3: AD11 -> /MC68040/TTL_AD20
- U100 pad P1: AD10 -> /MC68040/TTL_AD21
- U100 pad P16: SIZ1 -> /MC68040/TTL_SIZ1
- U100 pad P17: SIZ0 -> /MC68040/TTL_SIZ0
- U100 pad P2: TT1 -> /MC68040/TTL_TT1
- U100 pad P3: TT0 -> /MC68040/TTL_TT0
- U100 pad R15: TIP -> /MC68040/TTL_TIP
- U100 pad R16: TS -> /MC68040/TTL_TS
- U100 pad R3: RSTO -> /MC68040/TTL_RSTO
- U100 pad S13: TEA -> +5V
- U100 pad T11: AVEC -> +5V
- U100 pad T13: BG -> GND
- U100 pad T14: TA -> /MC68040/TTL_TA
- U100 pad T17: BB -> /MC68040/TTL_BB
- U100 pad T5: CDIS -> /MC68040/TTL_CDIS
- U100 pad T6: IPL2 -> /MC68040/TTL_IRQ
- U100 pad T7: IPL1 -> +5V
- U100 pad T8: IPL0 -> +5V
- U300 pad 2: AD0 -> +1V2
- U300 pad 3: AD16 -> +3V3
- U301 pad 1: GND -> /Power/AVR_RST
- U301 pad 10: +5V -> GND
- U301 pad 11: (no net) -> /Power/RST_SW
- U301 pad 12: DRAM_A0 -> /Power/PS_ON
- U301 pad 13: DRAM_A1 -> /Power/PWR_OK
- U301 pad 14: DRAM_A2 -> Net-(U301-Pad14)
- U301 pad 15: DRAM_A3 -> Net-(U301-Pad15)
- U301 pad 16: DRAM_A4 -> Net-(U301-Pad16)
- U301 pad 17: DRAM_A5 -> /Power/AVR_MOSI
- U301 pad 18: DRAM_A6 -> /Power/AVR_MISO
- U301 pad 19: DRAM_A10 -> /Power/AVR_SCK
- U301 pad 2: AD0 -> /Power/5V_IO0
- U301 pad 20: AD4 -> /Power/5VSB
- U301 pad 3: AD16 -> /Power/5V_IO1
- U301 pad 4: AD1 -> Net-(U301-Pad4)
- U301 pad 5: AD17 -> Net-(U301-Pad5)
- U301 pad 6: AD2 -> Net-(U301-Pad6)
- U301 pad 7: AD18 -> Net-(U301-Pad7)
- U301 pad 8: AD3 -> /Power/HDD_LED
- U301 pad 9: AD19 -> /Power/PWR_SW
Routing:
- net GND: track 0.00 -> 200.8 mm, vias 0 -> 132
- net ETH_INT: track 0.00 -> 180.6 mm, vias 0 -> 1
- net ETH_RST: track 0.00 -> 179.4 mm, vias 0 -> 1
- net PS2_CLK: track 0.00 -> 161.5 mm, vias 0 -> 1
- net PS2_DAT: track 0.00 -> 159.2 mm, vias 0 -> 1
- net ETH_CS: track 0.00 -> 151.8 mm, vias 0 -> 1
- net SD_CS: track 0.00 -> 148.2 mm
- net ETH_MOSI: track 0.00 -> 147.8 mm, vias 0 -> 1
- net ETH_SCK: track 0.00 -> 145.9 mm, vias 0 -> 1
- net SD_MOSI: track 0.00 -> 144.8 mm
- net SD_MISO: track 0.00 -> 143.7 mm
- net ETH_MISO: track 0.00 -> 142.6 mm, vias 0 -> 1
- net SD_SCK: track 0.00 -> 134.3 mm
- net +3V3: track 0.00 -> 130.8 mm, vias 0 -> 92
- net VGA_VSYNC: track 0.00 -> 125.9 mm, vias 0 -> 2
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- added copper zone on In2.Cu, net +1V2
- added copper zone on In2.Cu, net +3V3
- added copper zone on In2.Cu, net +5V
- added copper zone on In1.Cu, net GND
- removed copper zone on In1.Cu, net +5V
- removed copper zone on In2.Cu, net GND
Other:
- net class Clock added: clearance 0.127, trace_width 0.1468, via_dia 0.45, via_drill 0.2
- net class Default: clearance 0.1524 -> 0.127; trace_width 0.2 -> 0.127; via_dia 0.6 -> 0.45; via_drill 0.3 -> 0.2
- net class Power added: clearance 0.127, trace_width 0.254, via_dia 0.45, via_drill 0.2
- rule trace_clearance: 0.1524 -> 0.127
- rule trace_min: 0.2 -> 0.127
- rule via_min_drill: 0.3 -> 0.2
- rule via_min_size: 0.4 -> 0.45
- board text added: "3V3"
- board text added: "GND"
- board text added: "RXD"
- board text added: "TCK"
- board text added: "TDI"
- board text added: "TDO"
- board text added: "TMS"
- board text added: "TXD"
