File: cpu.sch (KiCad schematic (older format))
At the start: 2 parts, among them U100 MC68040RC, U102 W25Q80D

Commit message: Finished board + fab files
Parts:
- removed U102: W25Q80D, Package_SO:SOIC-8_3.9x4.9mm_P1.27mm, symbol winbond-nor:W25Q80D
- added C100, C101, C102, C103, C104, C105, C110, C111, C112, C113, C114, C115: 100nF, Capacitor_SMD:C_0603_1608Metric, symbol Device:C_Small
- added C116: 100uF, Capacitor_SMD:C_1206_3216Metric, symbol Device:C_Small
- added C117, C118: 4.7uF, Capacitor_SMD:C_0805_2012Metric, symbol Device:C_Small
- added R100: 4K7, Resistor_SMD:R_0603_1608Metric, symbol Device:R_Small
- added U110, U111, U120: MC74LCX16245, Package_SO:TSSOP-48_6.1x12.5mm_P0.5mm, symbol onsemi-buffer:MC74LCX16245
Connections:
- net AVEC is gone; now on net +5V: U100.T11 (~AVEC)
- net BG is gone; now on net GND: U100.T13 (~BG)
- net IPL0 is gone; now on net +5V: U100.T8 (~IPL0)
- net IPL1 is gone; now on net +5V: U100.T7 (~IPL1)
- net TEA is gone; now on net +5V: U100.S13 (~TEA)
- net +3V3: now also C100.1, C101.1, C102.1, C103.1, C104.1, C105.1, U110.18 (VCC), U110.31 (VCC), U110.42 (VCC), U110.7 (VCC), U111.18 (VCC), U111.31 (VCC), U111.42 (VCC), U111.7 (VCC), U120.1 (T/~R1), U120.18 (VCC), U120.31 (VCC), U120.42 (VCC), U120.7 (VCC)
- net +5V: now also C110.1, C111.1, C112.1, C113.1, C114.1, C115.1, C116.1, C117.1, C118.1, R100.1
- net AD0: now also U110.19 (B12); no longer U100.C3 (D0), U100.L18 (A0)
- net AD1: now also U110.20 (B13); no longer U100.B3 (D1), U100.K18 (A1)
- net AD10: now also U110.9 (B5); no longer U100.A8 (D10), U100.P1 (A10)
- net AD11: now also U110.8 (B4); no longer U100.A9 (D11), U100.N3 (A11)
- net AD12: now also U110.6 (B3); no longer U100.A10 (D12), U100.N1 (A12)
- net AD13: now also U110.5 (B2); no longer U100.A11 (D13), U100.M1 (A13)
- net AD14: now also U110.2 (B0); no longer U100.A12 (D14), U100.L1 (A14)
- net AD15: now also U111.22 (B14); no longer U100.A13 (D15), U100.K1 (A15)
- net AD16: now also U110.3 (B1); no longer U100.B11 (D16), U100.K2 (A16)
- net AD17: now also U111.20 (B13); no longer U100.A14 (D17), U100.J1 (A17)
- net AD18: now also U111.23 (B15); no longer U100.B12 (D18), U100.H1 (A18)
- net AD19: now also U111.17 (B11); no longer U100.A15 (D19), U100.J2 (A19)
- net AD2: now also U110.17 (B11); no longer U100.C4 (D2), U100.J17 (A2)
- net AD20: now also U111.13 (B8); no longer U100.A16 (D20), U100.G1 (A20)
- net AD21: now also U111.9 (B5); no longer U100.A17 (D21), U100.F1 (A21)
- net AD22: now also U111.14 (B9); no longer U100.B16 (D22), U100.E1 (A22)
- net AD23: now also U111.19 (B12); no longer U100.C15 (D23), U100.G3 (A23)
- net AD24: now also U111.6 (B3); no longer U100.A18 (D24), U100.D1 (A24)
- net AD25: now also U111.16 (B10); no longer U100.C16 (D25), U100.F3 (A25)
- net AD26: now also U111.5 (B2); no longer U100.B18 (D26), U100.E2 (A26)
- net AD27: now also U111.12 (B7); no longer U100.C1 (A27), U100.D16 (D27)
- net AD28: now also U111.3 (B1); no longer U100.C18 (D28), U100.E3 (A28)
- net AD29: now also U111.11 (B6); no longer U100.B1 (A29), U100.E16 (D29)
- net AD3: now also U110.23 (B15); no longer U100.A2 (D3), U100.J18 (A3)
- net AD30: now also U111.8 (B4); no longer U100.D3 (A30), U100.E17 (D30)
- net AD31: now also U111.2 (B0); no longer U100.A1 (A31), U100.D18 (D31)
- net AD4: now also U110.22 (B14); no longer U100.A3 (D4), U100.H18 (A4)
- net AD5: now also U110.16 (B10); no longer U100.A4 (D5), U100.G18 (A5)
- net AD6: now also U110.14 (B9); no longer U100.A5 (D6), U100.G16 (A6)
- net AD7: now also U110.13 (B8); no longer U100.A6 (D7), U100.F18 (A7)
- net AD8: now also U110.12 (B7); no longer U100.B7 (D8), U100.E18 (A8)
- net AD9: now also U110.11 (B6); no longer U100.A7 (D9), U100.F16 (A9)
- net CDIS: now also U120.16 (B10); no longer U100.T5 (~CDIS)
- net GND: now also C100.2, C101.2, C102.2, C103.2, C104.2, C105.2, C110.2, C111.2, C112.2, C113.2, C114.2, C115.2, C116.2, C117.2, C118.2, U110.10 (GND), U110.15 (GND), U110.21 (GND), U110.28 (GND), U110.34 (GND), U110.39 (GND), U110.4 (GND), U110.45 (GND), U111.10 (GND), U111.15 (GND), U111.21 (GND), U111.28 (GND), U111.34 (GND), U111.39 (GND), U111.4 (GND), U111.45 (GND), U120.10 (GND), U120.15 (GND), U120.21 (GND), U120.24 (T/~R2), U120.25 (~OE2), U120.28 (GND), U120.34 (GND), U120.39 (GND), U120.4 (GND), U120.45 (GND), U120.48 (~OE1)
- net RSTI: now also U120.17 (B11), U120.19 (B12), U120.20 (B13), U120.22 (B14), U120.23 (B15); no longer U100.S7 (~RSTI), U100.T3 (~TRST)
- net RSTO: now also U120.11 (B6); no longer U100.R3 (~RSTO)
- net RW: now also U120.2 (B0); no longer U100.N16 (R/~W)
- net SIZ0: now also U120.3 (B1); no longer U100.P17 (SIZ0)
- net SIZ1: now also U120.5 (B2); no longer U100.P16 (SIZ1)
- net TA: now also U120.13 (B8); no longer U100.T14 (~TA)
- net TIP: now also U120.8 (B4); no longer U100.R15 (~TIP)
- net TS: now also U120.6 (B3); no longer U100.R16 (~TS)
- net TT0: now also U120.9 (B5); no longer U100.P3 (TT0)
- net TT1: now also U120.12 (B7); no longer U100.P2 (TT1)
- net BB renamed TTL_BB
- net TTL_BB: now also R100.2
- net BR: no longer names the net of U100.T18 (~BR)
- net IPL2 renamed TTL_IRQ
- net TTL_IRQ: now also U120.35 (A9)
- net TM0: no longer names the net of U100.N18 (TM0)
- net TM1: no longer names the net of U100.M18 (TM1)
- net TM2: no longer names the net of U100.K17 (TM2)
- new net AD_DIR: U110.1 (T/~R1), U110.24 (T/~R2), U111.1 (T/~R1), U111.24 (T/~R2)
- new net AD_OE: U110.25 (~OE2), U110.48 (~OE1), U111.25 (~OE2), U111.48 (~OE1)
- new net IRQ: U120.14 (B9)
- new net TTL_AD0: U100.C3 (D0), U100.D1 (A24), U110.30 (A12)
- new net TTL_AD1: U100.B3 (D1), U100.C1 (A27), U110.29 (A13)
- new net TTL_AD10: U100.A8 (D10), U100.G1 (A20), U110.40 (A5)
- new net TTL_AD11: U100.A9 (D11), U100.G3 (A23), U110.41 (A4)
- new net TTL_AD12: U100.A10 (D12), U100.H1 (A18), U110.43 (A3)
- new net TTL_AD13: U100.A11 (D13), U100.J1 (A17), U110.44 (A2)
- new net TTL_AD14: U100.A12 (D14), U100.K1 (A15), U110.47 (A0)
- new net TTL_AD15: U100.A13 (D15), U100.L1 (A14), U111.27 (A14)
- new net TTL_AD16: U100.B11 (D16), U100.J2 (A19), U110.46 (A1)
- new net TTL_AD17: U100.A14 (D17), U100.M1 (A13), U111.29 (A13)
- new net TTL_AD18: U100.B12 (D18), U100.K2 (A16), U111.26 (A15)
- new net TTL_AD19: U100.A15 (D19), U100.N1 (A12), U111.32 (A11)
- new net TTL_AD2: U100.C4 (D2), U100.D3 (A30), U110.32 (A11)
- new net TTL_AD20: U100.A16 (D20), U100.N3 (A11), U111.36 (A8)
- new net TTL_AD21: U100.A17 (D21), U100.P1 (A10), U111.40 (A5)
- new net TTL_AD22: U100.B16 (D22), U100.K18 (A1), U111.35 (A9)
- new net TTL_AD23: U100.C15 (D23), U100.L18 (A0), U111.30 (A12)
- new net TTL_AD24: U100.A18 (D24), U100.J18 (A3), U111.43 (A3)
- new net TTL_AD25: U100.C16 (D25), U100.J17 (A2), U111.33 (A10)
- new net TTL_AD26: U100.B18 (D26), U100.H18 (A4), U111.44 (A2)
- new net TTL_AD27: U100.D16 (D27), U100.G16 (A6), U111.37 (A7)
- new net TTL_AD28: U100.C18 (D28), U100.G18 (A5), U111.46 (A1)
- new net TTL_AD29: U100.E16 (D29), U100.F16 (A9), U111.38 (A6)
- new net TTL_AD3: U100.A1 (A31), U100.A2 (D3), U110.26 (A15)
- new net TTL_AD30: U100.E17 (D30), U100.F18 (A7), U111.41 (A4)
- new net TTL_AD31: U100.D18 (D31), U100.E18 (A8), U111.47 (A0)
- new net TTL_AD4: U100.A3 (D4), U100.B1 (A29), U110.27 (A14)
- new net TTL_AD5: U100.A4 (D5), U100.E1 (A22), U110.33 (A10)
- new net TTL_AD6: U100.A5 (D6), U100.E2 (A26), U110.35 (A9)
- new net TTL_AD7: U100.A6 (D7), U100.E3 (A28), U110.36 (A8)
- new net TTL_AD8: U100.B7 (D8), U100.F1 (A21), U110.37 (A7)
- new net TTL_AD9: U100.A7 (D9), U100.F3 (A25), U110.38 (A6)
- new net TTL_CDIS: U100.T5 (~CDIS), U120.33 (A10)
- new net TTL_RSTI: U100.S7 (~RSTI), U100.T3 (~TRST), U120.32 (A11)
- new net TTL_RSTO: U100.R3 (~RSTO), U120.38 (A6)
- new net TTL_RW: U100.N16 (R/~W), U120.47 (A0)
- new net TTL_SIZ0: U100.P17 (SIZ0), U120.46 (A1)
- new net TTL_SIZ1: U100.P16 (SIZ1), U120.44 (A2)
- new net TTL_TA: U100.T14 (~TA), U120.36 (A8)
- new net TTL_TIP: U100.R15 (~TIP), U120.41 (A4)
- new net TTL_TS: U100.R16 (~TS), U120.43 (A3)
- new net TTL_TT0: U100.P3 (TT0), U120.40 (A5)
- new net TTL_TT1: U100.P2 (TT1), U120.37 (A7)
- no-connect marks 16 -> 24
Other:
- moved on the sheet: U100B, U100C, U100D
