File: pwr.sch (KiCad schematic (older format))
At the start: 1 part, among them J200 ATX20P

Commit message: Finished board + fab files
Parts:
- added C300, C301: 4.7uF, Capacitor_SMD:C_0805_2012Metric, symbol Device:C_Small
- added C302, C303, C304: 100nF, Capacitor_SMD:C_0603_1608Metric, symbol Device:C_Small
- added J301: PWR_SW, Connector_PinHeader_2.54mm:PinHeader_1x02_P2.54mm_Vertical, symbol Connector_Generic:Conn_01x02
- added J302: PWR_LED, Connector_PinHeader_2.54mm:PinHeader_1x02_P2.54mm_Vertical, symbol Connector_Generic:Conn_01x02
- added J303: RST_SW, Connector_PinHeader_2.54mm:PinHeader_1x02_P2.54mm_Vertical, symbol Connector_Generic:Conn_01x02
- added J304: HDD_LED, Connector_PinHeader_2.54mm:PinHeader_1x02_P2.54mm_Vertical, symbol Connector_Generic:Conn_01x02
- added J305: ISP, Connector_PinHeader_2.54mm:PinHeader_2x05_P2.54mm_Vertical, symbol Connector_Generic:Conn_02x05_Odd_Even
- added R300, R301, R302: 1K5, Resistor_SMD:R_0603_1608Metric, symbol Device:R_Small
- added U300: AZ1117-1.2, Package_TO_SOT_SMD:TO-252-2, symbol Regulator_Linear:AZ1117-1.2
- added U301: ATtiny2313A-PU, Package_DIP:DIP-20_W7.62mm, symbol MCU_Microchip_ATtiny:ATtiny2313A-PU
- added U302: TXB0102DCU, Package_SO:VSSOP-8_2.4x2.1mm_P0.5mm, symbol Logic_LevelTranslator:TXB0102DCU
- renumbered J200 to J300
Connections:
- net +3V3: now also C300.1, C304.1, U300.3 (VI), U302.3 (VCCA), U302.6 (OE)
- net +5V: now also R300.1
- net 5VSB: now also C302.1, C303.1, J305.2 (Pin_2), R302.1, U301.20 (VCC), U302.7 (VCCB)
- net GND: now also C300.2, C301.2, C302.2, C303.2, C304.2, J301.2 (Pin_2), J302.2 (Pin_2), J303.2 (Pin_2), J304.2 (Pin_2), J305.10 (Pin_10), J305.4 (Pin_4), J305.6 (Pin_6), J305.8 (Pin_8), U300.1 (GND), U301.10 (GND), U302.2 (GND)
- net PS_ON: now also U301.12 (PB0)
- net PWR_OK: now also U301.13 (PB1)
- new net: J302.1 (Pin_1), R300.2
- new net: J304.1 (Pin_1), R301.2
- new net +1V2: C301.1, U300.2 (VO)
- new net 5V_IO0: U301.2 (PD0), U302.8 (B1)
- new net 5V_IO1: U301.3 (PD1), U302.1 (B2)
- new net AVR_MISO: J305.9 (Pin_9), U301.18 (PB6)
- new net AVR_MOSI: J305.1 (Pin_1), U301.17 (PB5)
- new net AVR_RST: J305.5 (Pin_5), R302.2, U301.1 (PA2/~RESET)
- new net AVR_SCK: J305.7 (Pin_7), U301.19 (PB7)
- new net FPGA_IO0: U302.5 (A1)
- new net FPGA_IO1: U302.4 (A2)
- new net HDD_LED: R301.1, U301.8 (PD4)
- new net PWR_SW: J301.1 (Pin_1), U301.9 (PD5)
- new net RST_SW: J303.1 (Pin_1), U301.11 (PD6)
- no-connect marks 1 -> 9
